Commit message: :fire: New features & KEEPING LEARN gz_ros2_control !!!

File: drone_description/urdf/drone.urdf (robot description, URDF)
Before this commit: robot swarm_drone, 9 links, 8 joints
Links:
- removed link proppeller_BL_link
- removed link proppeller_BR_link
- removed link proppeller_FL_link
- removed link proppeller_FR_link
- added link propeller_BL_link, mass 0.05000; collision mesh filename=package://drone_description/meshes/collisions/prop_bl.stl scale=0.85046 0.75000 0.75000; visual mesh filename=package://drone_description/meshes/visuals/prop_bl.dae scale=0.85046 0.75000 0.75000
- added link propeller_BR_link, mass 0.05000; collision mesh filename=package://drone_description/meshes/collisions/prop_br.stl scale=0.75000 0.75000 0.75000; visual mesh filename=package://drone_description/meshes/visuals/prop_br.dae scale=0.75000 0.75000 0.75000
- added link propeller_FL_link, mass 0.05000; collision mesh filename=package://drone_description/meshes/collisions/prop_fl.stl scale=0.75000 0.75000 0.75000; visual mesh filename=package://drone_description/meshes/visuals/prop_fl.dae scale=0.75000 0.75000 0.75000
- added link propeller_FR_link, mass 0.05000; collision mesh filename=package://drone_description/meshes/collisions/prop_fl.stl scale=0.85046 0.75000 0.75000; visual mesh filename=package://drone_description/meshes/visuals/prop_fl.dae scale=0.85046 0.75000 0.75000
- link base_link: geometry collision mesh filename=package://drone_description/meshes/collisions/base.stl scale=1.00000 1.00000 1.00000; visual mesh filename=package://drone_description/meshes/visuals/base.dae scale=1.00000 1.00000 1.00000
- link camera_360_link: mass 0.12500 -> 0.03000; geometry collision mesh filename=package://drone_description/meshes/collisions/camera_360.stl scale=0.00072 0.00072 0.00072; visual mesh filename=package://drone_description/meshes/visuals/camera_360.dae scale=0.00072 0.00072 0.00072
- link camera_joint_1_link: mass 0.12500 -> 0.03000; geometry collision mesh filename=package://drone_description/meshes/collisions/camera_joint1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 scale=0.00072 0.00072 0.00072; visual mesh filename=package://drone_description/meshes/visuals/camera_joint1.dae scale=0.00072 0.00072 0.00072
- link camera_joint_2_link: mass 0.12500 -> 0.03000; geometry collision mesh filename=package://drone_description/meshes/collisions/camera_joint2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 scale=0.00072 0.00072 0.00072; visual mesh filename=package://drone_description/meshes/visuals/camera_joint2.dae scale=0.00072 0.00072 0.00072
- link depth_camera_link: mass 0.05000 -> 0.03100
Joints:
- removed joint proppeller_BL_link_joint
- removed joint proppeller_BR_link_joint
- removed joint proppeller_FL_link_joint
- removed joint proppeller_FR_link_joint
- added joint propeller_BL_link_joint: type continuous, parent base_link, child propeller_BL_link, origin xyz=0.18040 -0.17426 0.11755 rpy=0.00000 0.00000 0.00000, axis 0.00000 0.00000 1.00000, limit lower=0.00000 upper=0.00000 effort=0.00000 velocity=0.00000
- added joint propeller_BR_link_joint: type continuous, parent base_link, child propeller_BR_link, origin xyz=0.18040 0.17437 0.11755 rpy=0.00000 0.00000 0.00000, axis 0.00000 0.00000 -1.00000, limit lower=0.00000 upper=0.00000 effort=0.00000 velocity=0.00000
- added joint propeller_FL_link_joint: type continuous, parent base_link, child propeller_FL_link, origin xyz=-0.16748 -0.17426 0.11768 rpy=0.00000 0.00000 0.00000, axis 0.00000 0.00000 -1.00000, limit lower=0.00000 upper=0.00000 effort=0.00000 velocity=0.00000
- added joint propeller_FR_link_joint: type continuous, parent base_link, child propeller_FR_link, origin xyz=-0.16745 0.17390 0.11755 rpy=0.00000 0.00000 0.00000, axis 0.00000 0.00000 1.00000, limit lower=0.00000 upper=0.00000 effort=0.00000 velocity=0.00000
- joint camera_360_link_joint: origin xyz=0.00019 0.00002 -0.03339 rpy=2.21817 -1.57080 -0.61426 -> xyz=-0.00000 0.00000 -0.03433 rpy=2.53286 -1.57080 -0.94457; parent camera_joint_2_link -> camera_joint_1_link
- joint camera_joint_1_link_joint: origin xyz=0.01099 -0.00017 -0.01909 rpy=3.14159 -0.00000 -3.14159 -> xyz=-0.02297 0.00088 0.03900 rpy=2.75924 -1.57080 -2.79559; parent base_link -> camera_joint_2_link
- joint camera_joint_2_link_joint: origin xyz=-0.02223 0.00046 0.03019 rpy=2.77664 -1.57080 -2.79753 -> xyz=0.00665 -0.00026 -0.00516 rpy=3.14159 -0.00000 -3.14159; parent camera_joint_1_link -> base_link
- joint depth_camera_link_joint: origin xyz=-0.11887 -0.00145 0.07986 rpy=-0.00000 -0.00000 1.57080 -> xyz=-0.12089 0.00157 0.08506 rpy=0.00000 0.00000 1.57080
