Commit message: :fire: New features & KEEPING LEARN gz_ros2_control !!!

File: drone_description/urdf/drone.urdf.xacro (robot description, xacro)
@@ -6,103 +6,103 @@
   <link name="base_link">
     <collision name="base_collision">
+      <origin rpy="0.00000 0.00000 0.00000" xyz="0.00000 -0.00000 -0.00000"/>
+      <geometry>
+        <mesh filename="package://drone_description/meshes/collisions/base.stl" scale="1.00000 1.00000 1.00000"/>
+      </geometry>
+    </collision>
+    <inertial>
+      <inertia ixx="0.00558" ixy="-0.00000" ixz="0.00006" iyy="0.00469" iyz="0.00000" izz="0.00448"/>
+      <origin rpy="0.00000 0.00000 0.00000" xyz="0.00015 -0.00004 0.02583"/>
+      <mass value="0.32500"/>
+    </inertial>
+    <visual name="base">
+      <origin rpy="0.00000 0.00000 0.00000" xyz="0.00000 -0.00000 -0.00000"/>
+      <material name="Metal"/>
+      <geometry>
+        <mesh filename="package://drone_description/meshes/visuals/base.dae" scale="1.00000 1.00000 1.00000"/>
+      </geometry>
+    </visual>
+  </link>
+  <!-- Front left propeller link -->
+  <link name="propeller_FL_link">
+    <collision name="propeller_FL_collision">
+      <origin rpy="0.00000 0.00000 0.00000" xyz="0.00000 0.00000 0.00000"/>
+      <geometry>
+        <mesh filename="package://drone_description/meshes/collisions/prop_fl.stl" scale="0.75000 0.75000 0.75000"/>
+      </geometry>
+    </collision>
+    <inertial>
+      <inertia ixx="0.00006" ixy="0.00000" ixz="0.00000" iyy="0.00001" iyz="-0.00000" izz="0.00007"/>
       <origin rpy="0.00000 0.00000 0.00000" xyz="0.00000 -0.00000 0.00000"/>
-      <geometry>
-        <mesh filename="package://drone_description/meshes/collisions/base.stl" scale="0.00069 0.00069 0.00069"/>
-      </geometry>
-    </collision>
-    <inertial>
-      <inertia ixx="0.00557" ixy="-0.00000" ixz="0.00005" iyy="0.00469" iyz="0.00000" izz="0.00449"/>
-      <origin rpy="0.00000 0.00000 0.00000" xyz="-0.00011 -0.00005 0.02056"/>
-      <mass value="0.32500"/>
-    </inertial>
-    <visual name="base">
+      <mass value="0.05000"/>
+    </inertial>
+    <visual name="propeller_FL">
+      <origin rpy="0.00000 0.00000 0.00000" xyz="0.00000 0.00000 0.00000"/>
+      <material name="LandingRubber"/>
+      <geometry>
+        <mesh filename="package://drone_description/meshes/visuals/prop_fl.dae" scale="0.75000 0.75000 0.75000"/>
+      </geometry>
+    </visual>
+  </link>
+  <!-- Front left propeller link -->
+  <link name="propeller_FR_link">
+    <collision name="propeller_FR_collision">
+      <origin rpy="0.00000 0.00000 0.00000" xyz="0.00000 0.00000 -0.00000"/>
+      <geometry>
+        <mesh filename="package://drone_description/meshes/collisions/prop_fl.stl" scale="0.85046 0.75000 0.75000"/>
+      </geometry>
+    </collision>
+    <inertial>
+      <inertia ixx="0.00006" ixy="-0.00000" ixz="-0.00000" iyy="0.00001" iyz="0.00000" izz="0.00007"/>
+      <origin rpy="0.00000 0.00000 0.00000" xyz="-0.00000 -0.00000 -0.00000"/>
+      <mass value="0.05000"/>
+    </inertial>
+    <visual name="propeller_FR">
+      <origin rpy="0.00000 0.00000 0.00000" xyz="0.00000 -0.00000 -0.00000"/>
+      <material name="LandingRubber"/>
+      <geometry>
+        <mesh filename="package://drone_description/meshes/visuals/prop_fl.dae" scale="0.85046 0.75000 0.75000"/>
+      </geometry>
+    </visual>
+  </link>
+  <!-- Back left propeller link -->
+  <link name="propeller_BL_link">
+    <collision name="propeller_BL_collision">
+      <origin rpy="0.00000 0.00000 0.00000" xyz="0.00000 0.00000 -0.00000"/>
+      <geometry>
+        <mesh filename="package://drone_description/meshes/collisions/prop_bl.stl" scale="0.85046 0.75000 0.75000"/>
+      </geometry>
+    </collision>
+    <inertial>
+      <inertia ixx="0.00006" ixy="-0.00000" ixz="-0.00000" iyy="0.00001" iyz="0.00000" izz="0.00007"/>
+      <origin rpy="0.00000 0.00000 0.00000" xyz="-0.00000 -0.00000 -0.00000"/>
+      <mass value="0.05000"/>
+    </inertial>
+    <visual name="propeller_BL">
+      <origin rpy="0.00000 0.00000 0.00000" xyz="0.00000 0.00000 0.00000"/>
+      <material name="LandingRubber"/>
+      <geometry>
+        <mesh filename="package://drone_description/meshes/visuals/prop_bl.dae" scale="0.85046 0.75000 0.75000"/>
+      </geometry>
+    </visual>
+  </link>
+  <!-- Back right propeller link -->
+  <link name="propeller_BR_link">
+    <collision name="propeller_BR_collision">
+      <origin rpy="0.00000 0.00000 0.00000" xyz="0.00000 -0.00000 -0.00000"/>
+      <geometry>
+        <mesh filename="package://drone_description/meshes/collisions/prop_br.stl" scale="0.75000 0.75000 0.75000"/>
+      </geometry>
+    </collision>
+    <inertial>
+      <inertia ixx="0.00006" ixy="0.00000" ixz="0.00000" iyy="0.00001" iyz="-0.00000" izz="0.00007"/>
+      <origin rpy="0.00000 0.00000 0.00000" xyz="-0.00000 -0.00000 -0.00000"/>
+      <mass value="0.05000"/>
+    </inertial>
+    <visual name="propeller_BR">
       <origin rpy="0.00000 0.00000 0.00000" xyz="0.00000 -0.00000 0.00000"/>
       <material name="LandingRubber"/>
       <geometry>
-        <mesh filename="package://drone_description/meshes/visuals/base.dae" scale="0.00069 0.00069 0.00069"/>
-      </geometry>
-    </visual>
-  </link>
-  <!-- Front left proppeller link -->
-  <link name="proppeller_FL_link">
-    <collision name="proppeller_FL_collision">
-      <origin rpy="1.57080 -0.00000 0.00000" xyz="-0.00000 -0.00000 -0.00000"/>
-      <geometry>
-        <mesh filename="package://drone_description/meshes/collisions/prop_fl.stl" scale="0.01000 0.01000 0.01000"/>
-      </geometry>
-    </collision>
-    <inertial>
-      <inertia ixx="0.00007" ixy="0.00000" ixz="0.00000" iyy="0.00001" iyz="-0.00000" izz="0.00007"/>
-      <origin rpy="0.00000 0.00000 0.00000" xyz="-0.00000 -0.00000 -0.00000"/>
-      <mass value="0.05000"/>
-    </inertial>
-    <visual name="proppeller_FL">
-      <origin rpy="1.57080 -0.00000 0.00000" xyz="-0.00000 -0.00000 -0.00000"/>
-      <material name="green_metal"/>
-      <geometry>
-        <mesh filename="package://drone_description/meshes/visuals/prop_fl.dae" scale="0.01000 0.01000 0.01000"/>
-      </geometry>
-    </visual>
-  </link>
-  <!-- Front right proppeller link -->
-  <link name="proppeller_FR_link">
-    <collision name="proppeller_FR_collision">
-      <origin rpy="1.57080 -0.00000 0.00000" xyz="0.00000 0.00000 -0.00000"/>
-      <geometry>
-        <mesh filename="package://drone_description/meshes/collisions/prop_fr.stl" scale="0.01000 0.01000 0.01000"/>
-      </geometry>
-    </collision>
-    <inertial>
-      <inertia ixx="0.00007" ixy="-0.00000" ixz="0.00000" iyy="0.00001" iyz="0.00000" izz="0.00007"/>
-      <origin rpy="0.00000 0.00000 0.00000" xyz="0.00000 0.00000 -0.00000"/>
-      <mass value="0.05000"/>
-    </inertial>
-    <visual name="proppeller_FR">
-      <origin rpy="1.57080 -0.00000 0.00000" xyz="-0.00000 0.00000 -0.00000"/>
-      <material name="green_metal"/>
-      <geometry>
-        <mesh filename="package://drone_description/meshes/visuals/prop_fr.dae" scale="0.01000 0.01000 0.01000"/>
-      </geometry>
-    </visual>
-  </link>
-  <!-- Back left proppeller link -->
-  <link name="proppeller_BL_link">
-    <collision name="proppeller_BL_collision">
-      <origin rpy="1.57080 0.00000 0.00000" xyz="0.00000 -0.00000 -0.00000"/>
-      <geometry>
-        <mesh filename="package://drone_description/meshes/collisions/prop_bl.stl" scale="0.01000 0.01000 0.01000"/>
-      </geometry>
-    </collision>
-    <inertial>
-      <inertia ixx="0.00007" ixy="-0.00000" ixz="-0.00000" iyy="0.00001" iyz="-0.00000" izz="0.00007"/>
-      <origin rpy="0.00000 0.00000 0.00000" xyz="0.00000 -0.00000 -0.00000"/>
-      <mass value="0.05000"/>
-    </inertial>
-    <visual name="proppeller_BL">
-      <origin rpy="1.57080 0.00000 0.00000" xyz="0.00000 -0.00000 -0.00000"/>
-      <material name="green_metal"/>
-      <geometry>
-        <mesh filename="package://drone_description/meshes/visuals/prop_bl.dae" scale="0.01000 0.01000 0.01000"/>
-      </geometry>
-    </visual>
-  </link>
-  <!-- Back right proppeller link -->
-  <link name="proppeller_BR_link">
-    <collision name="proppeller_BR_collision">
-      <origin rpy="1.57080 0.00000 0.00000" xyz="-0.00000 -0.00000 -0.00000"/>
-      <geometry>
-        <mesh filename="package://drone_description/meshes/collisions/prop_br.stl" scale="0.01000 0.01000 0.01000"/>
-      </geometry>
-    </collision>
-    <inertial>
-      <inertia ixx="0.00007" ixy="0.00000" ixz="-0.00000" iyy="0.00001" iyz="-0.00000" izz="0.00007"/>
-      <origin rpy="0.00000 0.00000 0.00000" xyz="-0.00000 -0.00000 -0.00000"/>
-      <mass value="0.05000"/>
-    </inertial>
-    <visual name="proppeller_BR">
-      <origin rpy="1.57080 0.00000 0.00000" xyz="-0.00000 -0.00000 -0.00000"/>
-      <material name="green_metal"/>
-      <geometry>
-        <mesh filename="package://drone_description/meshes/visuals/prop_br.dae" scale="0.01000 0.01000 0.01000"/>
+        <mesh filename="package://drone_description/meshes/visuals/prop_br.dae" scale="0.75000 0.75000 0.75000"/>
       </geometry>
     </visual>
@@ -110,31 +110,20 @@
   <!-- Camera 360 link -->
   <link name="camera_360_link">
-    <sensor name="camera_360" type="camera">
-      <origin rpy="1.55815 -1.48401 -1.52510" xyz="-0.02318 0.00259 -0.00057"/>
-      <parent link="camera_360_link"/>
-      <camera>
-        <image>
-          <width>640</width>
-          <height>480</height>
-          <hfov>1.57080</hfov>
-        </image>
-      </camera>
-    </sensor>
     <collision name="camera_360_collision">
-      <origin rpy="-1.67352 -0.01991 -0.11320" xyz="0.00062 0.00343 -0.00033"/>
-      <geometry>
-        <mesh filename="package://drone_description/meshes/collisions/camera_360.stl" scale="0.00069 0.00069 0.00069"/>
-      </geometry>
-    </collision>
-    <inertial>
-      <inertia ixx="0.00002" ixy="-0.00000" ixz="-0.00000" iyy="0.00003" iyz="-0.00000" izz="0.00003"/>
-      <origin rpy="0.00000 0.00000 0.00000" xyz="-0.00276 -0.00079 0.00002"/>
-      <mass value="0.12500"/>
+      <origin rpy="-1.57080 0.00000 -0.11900" xyz="-0.00000 -0.00000 0.00000"/>
+      <geometry>
+        <mesh filename="package://drone_description/meshes/collisions/camera_360.stl" scale="0.00072 0.00072 0.00072"/>
+      </geometry>
+    </collision>
+    <inertial>
+      <inertia ixx="0.00001" ixy="-0.00000" ixz="-0.00000" iyy="0.00001" iyz="-0.00000" izz="0.00001"/>
+      <origin rpy="0.00000 0.00000 0.00000" xyz="-0.00243 -0.00074 -0.00000"/>
+      <mass value="0.03000"/>
     </inertial>
     <visual name="camera_360">
-      <origin rpy="-1.67352 -0.01991 -0.11320" xyz="0.00062 0.00343 -0.00033"/>
-      <material name="RailsRubber"/>
-      <geometry>
-        <mesh filename="package://drone_description/meshes/visuals/camera_360.dae" scale="0.00069 0.00069 0.00069"/>
+      <origin rpy="-1.57080 0.00000 -0.11900" xyz="-0.00000 -0.00000 0.00000"/>
+      <material name="Metal"/>
+      <geometry>
+        <mesh filename="package://drone_description/meshes/visuals/camera_360.dae" scale="0.00072 0.00072 0.00072"/>
       </geometry>
     </visual>
@@ -143,19 +132,19 @@
   <link name="camera_joint_1_link">
     <collision name="camera_joint_1_collision">
-      <origin rpy="3.14159 0.00000 -3.14159" xyz="-0.03933 -0.00000 0.01897"/>
-      <geometry>
-        <mesh filename="package://drone_description/meshes/collisions/camera_joint1.stl" scale="0.00069 0.00069 0.00069"/>
-      </geometry>
-    </collision>
-    <inertial>
-      <inertia ixx="0.00100" ixy="0.00000" ixz="0.00000" iyy="0.00100" iyz="0.00000" izz="0.00100"/>
-      <origin rpy="0.00000 0.00000 0.00000" xyz="0.00000 0.00000 -0.00000"/>
-      <mass value="0.12500"/>
+    <origin rpy="0.66577 -1.57080 -0.64827" xyz="-0.00000 0.00000 0.00000"/>
+      <geometry>
+        <mesh filename="package://drone_description/meshes/collisions/camera_joint1.stl" scale="0.00072 0.00072 0.00072"/>
+      </geometry>
+    </collision>
+    <inertial>
+      <inertia ixx="0.00001" ixy="-0.00000" ixz="0.00000" iyy="0.00001" iyz="-0.00000" izz="0.00001"/>
+      <origin rpy="0.00000 0.00000 0.00000" xyz="-0.00002 -0.00019 -0.01854"/>
+      <mass value="0.03000"/>
     </inertial>
     <visual name="camera_joint_1">
-      <origin rpy="3.14159 0.00000 3.12071" xyz="-0.03932 0.00082 0.01897"/>
-      <material name="RailsAntennaHolder"/>
-      <geometry>
-        <mesh filename="package://drone_description/meshes/visuals/camera_joint1.dae" scale="0.00069 0.00069 0.00069"/>
+      <origin rpy="0.66577 -1.57080 -0.64827" xyz="-0.00000 0.00000 0.00000"/>
+      <material name="Material.005"/>
+      <geometry>
+        <mesh filename="package://drone_description/meshes/visuals/camera_joint1.dae" scale="0.00072 0.00072 0.00072"/>
       </geometry>
     </visual>
@@ -164,19 +153,19 @@
   <link name="camera_joint_2_link">
     <collision name="camera_joint_2_collision">
-      <origin rpy="1.57078 -1.54991 -1.57078" xyz="0.00022 0.00039 -0.01975"/>
-      <geometry>
-        <mesh filename="package://drone_description/meshes/collisions/camera_joint2.stl" scale="0.00069 0.00069 0.00069"/>
-      </geometry>
-    </collision>
-    <inertial>
-      <inertia ixx="0.00004" ixy="-0.00000" ixz="0.00000" iyy="0.00002" iyz="-0.00000" izz="0.00005"/>
-      <origin rpy="0.00000 0.00000 0.00000" xyz="0.00027 -0.00019 -0.01827"/>
-      <mass value="0.12500"/>
+    <origin rpy="3.14159 0.00000 3.10524" xyz="0.00000 -0.00000 -0.00000"/>
+      <geometry>
+        <mesh filename="package://drone_description/meshes/collisions/camera_joint2.stl" scale="0.00072 0.00072 0.00072"/>
+      </geometry>
+    </collision>
+    <inertial>
+      <inertia ixx="0.000001" ixy="0" ixz="0" iyy="0.000001" iyz="0" izz="0.000001"/>
+      <origin rpy="0.00000 0.00000 0.00000" xyz="-0.02035 -0.00003 0.01431"/>
+      <mass value="0.03000"/>
     </inertial>
     <visual name="camera_joint_2">
-      <origin rpy="0.66324 -1.57080 -0.63013" xyz="0.00021 0.00045 -0.01976"/>
-      <material name="Metal"/>
-      <geometry>
-        <mesh filename="package://drone_description/meshes/visuals/camera_joint2.dae" scale="0.00069 0.00069 0.00069"/>
+      <origin rpy="3.14159 0.00000 3.10524" xyz="0.00000 -0.00000 -0.00000"/>
+      <material name="RailsAntennaHolder"/>
+      <geometry>
+        <mesh filename="package://drone_description/meshes/visuals/camera_joint2.dae" scale="0.00072 0.00072 0.00072"/>
       </geometry>
     </visual>
@@ -184,17 +173,6 @@
   <!-- Depth camera link -->
   <link name="depth_camera_link">
-    <sensor name="depth_camera" type="camera">
-      <origin rpy="-1.57080 0.00000 0.00000" xyz="0.00000 0.00736 0.00000"/>
-      <parent link="depth_camera_link"/>
-      <camera>
-        <image>
-          <width>640</width>
-          <height>480</height>
-          <hfov>1.57080</hfov>
-        </image>
-      </camera>
-    </sensor>
     <collision name="depth_camera_collision">
-      <origin rpy="1.57080 0.00000 0.00000" xyz="0.00000 -0.00000 -0.00000"/>
+      <origin rpy="0.00000 0.00000 0.00000" xyz="-0.00000 0.00000 0.00000"/>
       <geometry>
         <mesh filename="package://drone_description/meshes/collisions/depth_camera.stl" scale="0.01000 0.01000 0.01000"/>
@@ -202,11 +180,11 @@
     </collision>
     <inertial>
-      <inertia ixx="0.00003" ixy="-0.00000" ixz="0.00000" iyy="0.00000" iyz="-0.00000" izz="0.00003"/>
-      <origin rpy="0.00000 0.00000 0.00000" xyz="0.00000 -0.00000 -0.00000"/>
-      <mass value="0.05000"/>
+      <inertia ixx="0.00002" ixy="-0.00000" ixz="0.00000" iyy="0.00000" iyz="-0.00000" izz="0.00002"/>
+      <origin rpy="0.00000 0.00000 0.00000" xyz="-0.00019 -0.00127 -0.00001"/>
+      <mass value="0.03100"/>
     </inertial>
     <visual name="depth_camera">
-      <origin rpy="1.57080 -0.00000 0.00000" xyz="0.00000 -0.00000 -0.00000"/>
-      <material name="CameraMesh.003"/>
+      <origin rpy="0.00000 0.00000 0.00000" xyz="-0.00000 0.00000 0.00000"/>
+      <material name="CameraMesh.001"/>
       <geometry>
         <mesh filename="package://drone_description/meshes/visuals/depth_camera.dae" scale="0.01000 0.01000 0.01000"/>
@@ -214,41 +192,41 @@
     </visual>
   </link>
-  <!-- Proppeller front left joint -->
-  <joint name="proppeller_BL_link_joint" type="continuous">
-    <limit lower="0.00000" upper="0.00000" effort="0.00000" velocity="0.00000"/>
-    <origin rpy="0.00000 0.00000 -0.00000" xyz="0.18070 -0.17501 0.11613"/>
-    <parent link="base_link"/>
-    <child link="proppeller_BL_link"/>
-    <axis xyz="0.00000 0.00000 1.00000"/>
-  </joint>
-  <!-- Proppeller front right joint -->
-  <joint name="proppeller_BR_link_joint" type="continuous">
-    <limit lower="0.00000" upper="0.00000" effort="0.00000" velocity="0.00000"/>
-    <origin rpy="0.00000 0.00000 -0.00000" xyz="0.18070 0.17477 0.11613"/>
-    <parent link="base_link"/>
-    <child link="proppeller_BR_link"/>
+  <!-- Propeller front left joint -->
+  <joint name="propeller_FL_link_joint" type="continuous">
+    <limit lower="0.00000" upper="0.00000" effort="0.00000" velocity="0.00000"/>
+    <origin rpy="0.00000 0.00000 0.00000" xyz="-0.16748 -0.17426 0.11768"/>
+    <parent link="base_link"/>
+    <child link="propeller_FL_link"/>
     <axis xyz="0.00000 0.00000 -1.00000"/>
   </joint>
-  <!-- Proppeller back left joint -->
-  <joint name="proppeller_FL_link_joint" type="continuous">
-    <limit lower="0.00000" upper="0.00000" effort="0.00000" velocity="0.00000"/>
-    <origin rpy="0.00000 0.00000 -0.00000" xyz="-0.16902 -0.17494 0.11613"/>
-    <parent link="base_link"/>
-    <child link="proppeller_FL_link"/>
+  <!-- Propeller front right joint -->
+  <joint name="propeller_FR_link_joint" type="continuous">
+    <limit lower="0.00000" upper="0.00000" effort="0.00000" velocity="0.00000"/>
+    <origin rpy="0.00000 0.00000 0.00000" xyz="-0.16745 0.17390 0.11755"/>
+    <parent link="base_link"/>
+    <child link="propeller_FR_link"/>
+    <axis xyz="0.00000 0.00000 1.00000"/>
+  </joint>
+  <!-- Propeller back left joint -->
+  <joint name="propeller_BL_link_joint" type="continuous">
+    <limit lower="0.00000" upper="0.00000" effort="0.00000" velocity="0.00000"/>
+    <origin rpy="0.00000 0.00000 0.00000" xyz="0.18040 -0.17426 0.11755"/>
+    <parent link="base_link"/>
+    <child link="propeller_BL_link"/>
+    <axis xyz="0.00000 0.00000 1.00000"/>
+  </joint>
+  <!-- Propeller back right joint -->
+  <joint name="propeller_BR_link_joint" type="continuous">
+    <limit lower="0.00000" upper="0.00000" effort="0.00000" velocity="0.00000"/>
+    <origin rpy="0.00000 0.00000 0.00000" xyz="0.18040 0.17437 0.11755"/>
+    <parent link="base_link"/>
+    <child link="propeller_BR_link"/>
     <axis xyz="0.00000 0.00000 -1.00000"/>
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
File: drone_description/urdf/materials_and_colors.xacro (robot description, xacro)
@@ -1,7 +1,13 @@
 <?xml version="1.0" encoding="utf-8"?>
 <robot xmlns:xacro="http://www.ros.org/wiki/xacro">
+  <material name="CameraMesh.001">
+    <color rgba="0.02745 0.02745 0.02745 1.00000"/>
+  </material>
   <!-- Dark grey color for the depth camera plastic material -->
   <material name="CameraMesh.003">
     <color rgba="0.02745 0.02745 0.02745 1.00000"/>
+  </material>
+  <material name="Material.005">
+    <color rgba="0.80000 0.80000 0.80000 1.00000"/>
   </material>
   <!-- Darker black color for the landing drone parts -->
@@ -25,3 +31,8 @@
     <color rgba="0.10048 0.10048 0.10048 1.00000"/>
   </material>
+  <!-- Fiber carbon material for the drone -->
+  <material name="CarbonFiber">
+    <texture filename="package://drone_description/meshes/visuals/CF.png"/>
+    <color rgba="0.80000 0.80000 0.80000 1.00000"/>
+  </material>
 </robot>

Commit message: 🤖✨ Comprehensive update to robotics packages
🔧 Configuration:
- Adjusted controllers for Gazebo Harmonic with ROS 2.

📦 Models:
- Enhanced and updated URDF/SDF files for the X500 drone.
- Optimized physical and visual parameters of the model.

📡 Communication:
- Integrated topics and services for ROS 2.

🔍 Improvements:
- Refactored simulation parameters and controllers.
- Simplified file paths and folder organization.

🌟 Miscellaneous:
- Added basic documentation for custom configurations.

File: drone_description/urdf/drone.urdf (robot description, URDF)
Before this commit: robot swarm_drone, 9 links, 8 joints
Links:
- link propeller_FR_link: geometry collision mesh filename=package://drone_description/meshes/collisions/prop_fr.stl scale=0.85046 0.75000 0.75000; visual mesh filename=package://drone_description/meshes/visuals/prop_fr.dae scale=0.85046 0.75000 0.75000

File: drone_description/urdf/drone.urdf.xacro (robot description, xacro)
@@ -45,10 +45,10 @@
     </visual>
   </link>
-  <!-- Front left propeller link -->
+  <!-- Front right propeller link -->
   <link name="propeller_FR_link">
     <collision name="propeller_FR_collision">
       <origin rpy="0.00000 0.00000 0.00000" xyz="0.00000 0.00000 -0.00000"/>
       <geometry>
-        <mesh filename="package://drone_description/meshes/collisions/prop_fl.stl" scale="0.85046 0.75000 0.75000"/>
+        <mesh filename="package://drone_description/meshes/collisions/prop_fr.stl" scale="0.85046 0.75000 0.75000"/>
       </geometry>
     </collision>
@@ -62,5 +62,5 @@
       <material name="LandingRubber"/>
       <geometry>
-        <mesh filename="package://drone_description/meshes/visuals/prop_fl.dae" scale="0.85046 0.75000 0.75000"/>
+        <mesh filename="package://drone_description/meshes/visuals/prop_fr.dae" scale="0.85046 0.75000 0.75000"/>
       </geometry>
     </visual>

File: drone_description/urdf/drone_gazebo_controllers.xacro (robot description, xacro)
@@ -2,5 +2,5 @@
 <robot xmlns:xacro="http://www.ros.org/wiki/xacro">
   <!-- ROS 2 Control Configuration -->
-  <ros2_control name="DroneControl" type="system">
+  <ros2_control name="GazeboSimSystem" type="system">
     <hardware>
       <plugin>gz_ros2_control/GazeboSimSystem</plugin>
