Commit message: 🚀 feat(urdf): Complete Gazebo physics overhaul
✨ Changed:
- 🎨 Converted all materials to Gazebo-specific definitions (#MaterialFix)
- ⚙️ Updated friction model to Gazebo Sim (Ignition) syntax (#PhysicsUpdate)
- 📦 Added proper collision surface parameters for all components
- 🛠️ Fixed texture paths and material references in visual meshes

🔧 Adjusted:
- 🛑 Friction coefficients (μ/μ2) for different materials:
  • 🤖 Base: 0.5/0.4 (hard plastic)
  • 🛩️ Propellers: 1.5/1.2 (high-friction rubber)
  • 📷 Camera joints: 0.3/0.2 (polished metal)
  • 🔭 Sensors: 0.8/0.6 (dark plastic)
- 🧮 Contact physics (kp/kd) for realistic collisions
- 🎮 Control plugin path to use ROS2 package variables

➕ Added:
- 💡 Material fallback system for missing textures
- 🌐 Wildcard selector for multi-component materials
- 📝 Detailed physics comments for each component
- 🔄 Directional friction model template (fdir1)

🐛 Fixed:
- 🚫 Removed deprecated <mu1>/<mu2> syntax
- 🔗 Corrected collision reference frames
- 🖼️ Texture loading issues with proper .material file setup

📚 Documentation:
- 📌 Added Gazebo resource path instructions
- 💡 Physics parameter explanations in comments

File: drone_description/urdf/drone.urdf.xacro (robot description, xacro)
@@ -1,6 +1,4 @@
 <?xml version="1.0" encoding="utf-8"?>
 <robot xmlns:xacro="http://www.ros.org/wiki/xacro" name="swarm_drone">
-  <!-- Include the materials and colors -->
-  <xacro:include filename="$(find drone_description)/urdf/materials_and_colors.xacro"/>
   <!-- Main quadcopter link -->
   <link name="base_link">
@@ -18,5 +16,4 @@
     <visual name="base">
       <origin rpy="0.00000 0.00000 0.00000" xyz="0.00000 -0.00000 -0.00000"/>
-      <material name="Metal"/>
       <geometry>
         <mesh filename="package://drone_description/meshes/visuals/base.dae" scale="1.00000 1.00000 1.00000"/>
@@ -39,5 +36,4 @@
     <visual name="propeller_FL">
       <origin rpy="0.00000 0.00000 0.00000" xyz="0.00000 0.00000 0.00000"/>
-      <material name="LandingRubber"/>
       <geometry>
         <mesh filename="package://drone_description/meshes/visuals/prop_fl.dae" scale="0.75000 0.75000 0.75000"/>
@@ -60,5 +56,4 @@
     <visual name="propeller_FR">
       <origin rpy="0.00000 0.00000 0.00000" xyz="0.00000 -0.00000 -0.00000"/>
-      <material name="LandingRubber"/>
       <geometry>
         <mesh filename="package://drone_description/meshes/visuals/prop_fr.dae" scale="0.85046 0.75000 0.75000"/>
@@ -81,5 +76,4 @@
     <visual name="propeller_BL">
       <origin rpy="0.00000 0.00000 0.00000" xyz="0.00000 0.00000 0.00000"/>
-      <material name="LandingRubber"/>
       <geometry>
         <mesh filename="package://drone_description/meshes/visuals/prop_bl.dae" scale="0.85046 0.75000 0.75000"/>
@@ -102,5 +96,4 @@
     <visual name="propeller_BR">
       <origin rpy="0.00000 0.00000 0.00000" xyz="0.00000 -0.00000 0.00000"/>
-      <material name="LandingRubber"/>
       <geometry>
         <mesh filename="package://drone_description/meshes/visuals/prop_br.dae" scale="0.75000 0.75000 0.75000"/>
@@ -123,5 +116,4 @@
     <visual name="camera_360">
       <origin rpy="-1.57080 0.00000 -0.11900" xyz="-0.00000 -0.00000 0.00000"/>
-      <material name="Metal"/>
       <geometry>
         <mesh filename="package://drone_description/meshes/visuals/camera_360.dae" scale="0.00072 0.00072 0.00072"/>
@@ -144,5 +136,4 @@
     <visual name="camera_joint_1">
       <origin rpy="0.66577 -1.57080 -0.64827" xyz="-0.00000 0.00000 0.00000"/>
-      <material name="Material.005"/>
       <geometry>
         <mesh filename="package://drone_description/meshes/visuals/camera_joint1.dae" scale="0.00072 0.00072 0.00072"/>
@@ -165,5 +156,4 @@
     <visual name="camera_joint_2">
       <origin rpy="3.14159 0.00000 3.10524" xyz="0.00000 -0.00000 -0.00000"/>
-      <material name="RailsAntennaHolder"/>
       <geometry>
         <mesh filename="package://drone_description/meshes/visuals/camera_joint2.dae" scale="0.00072 0.00072 0.00072"/>
@@ -186,5 +176,4 @@
     <visual name="depth_camera">
       <origin rpy="0.00000 0.00000 0.00000" xyz="-0.00000 0.00000 0.00000"/>
-      <material name="CameraMesh.001"/>
       <geometry>
         <mesh filename="package://drone_description/meshes/visuals/depth_camera.dae" scale="0.01000 0.01000 0.01000"/>
@@ -254,4 +243,6 @@
     <child link="depth_camera_link"/>
   </joint>
+  <!-- Include the gazebo materials -->
+  <xacro:include filename="$(find drone_description)/urdf/gazebo_materials.xacro"/>
   <!-- Include the gazebo controllers -->
   <xacro:include filename="$(find drone_description)/urdf/drone_gazebo_controllers.xacro"/>

Commit message: 🔧🔄🚁 Finalize drone physics and controller config for Gazebo simulation
- ✨ Changed propeller joints to `continuous` type (proper 360° rotation)
- 🗑️ Removed invalid angular limits (`lower`/`upper`) from continuous joints
- 📉 Set realistic motor constraints:
  - Max torque: 0.3 Nm (X500-equivalent brushless motors)
  - Max velocity: 314.16 rad/s ≜ 3000 RPM (industry-standard for 10" props)
- 🎯 Fixed camera joints interface mismatch:
  - 📸 Switched to position control for revolute joints
  - 🔄 Added smooth position constraints (0.5° tolerance)
- ⚡ Simplified ros2_control config:
  - Removed redundant effort interfaces from camera joints
  - Standardized command interfaces across controllers

File: drone_description/urdf/drone.urdf.xacro (robot description, xacro)
@@ -183,5 +183,5 @@
   <!-- Propeller front left joint -->
   <joint name="propeller_FL_link_joint" type="continuous">
-    <limit lower="0.00000" upper="0.00000" effort="0.00000" velocity="0.00000"/>
+    <limit effort="0.3" velocity="314.16"/>
     <origin rpy="0.00000 0.00000 0.00000" xyz="-0.16748 -0.17426 0.11768"/>
     <parent link="base_link"/>
@@ -191,5 +191,5 @@
   <!-- Propeller front right joint -->
   <joint name="propeller_FR_link_joint" type="continuous">
-    <limit lower="0.00000" upper="0.00000" effort="0.00000" velocity="0.00000"/>
+    <limit effort="0.3" velocity="314.16"/>
     <origin rpy="0.00000 0.00000 0.00000" xyz="-0.16745 0.17390 0.11755"/>
     <parent link="base_link"/>
@@ -199,5 +199,5 @@
   <!-- Propeller back left joint -->
   <joint name="propeller_BL_link_joint" type="continuous">
-    <limit lower="0.00000" upper="0.00000" effort="0.00000" velocity="0.00000"/>
+    <limit effort="0.3" velocity="314.16"/>
     <origin rpy="0.00000 0.00000 0.00000" xyz="0.18040 -0.17426 0.11755"/>
     <parent link="base_link"/>
@@ -207,5 +207,5 @@
   <!-- Propeller back right joint -->
   <joint name="propeller_BR_link_joint" type="continuous">
-    <limit lower="0.00000" upper="0.00000" effort="0.00000" velocity="0.00000"/>
+    <limit effort="0.3" velocity="314.16"/>
     <origin rpy="0.00000 0.00000 0.00000" xyz="0.18040 0.17437 0.11755"/>
     <parent link="base_link"/>
@@ -215,5 +215,5 @@
   <!-- Camera 360 joint -->
   <joint name="camera_360_link_joint" type="revolute">
-    <limit lower="-3.14000" upper="3.14000" effort="0.00000" velocity="0.00000"/>
+    <limit lower="-3.14000" upper="3.14000" effort="10.0" velocity="3.14"/>
     <origin rpy="2.53286 -1.57080 -0.94457" xyz="-0.00000 0.00000 -0.03433"/>
     <parent link="camera_joint_1_link"/>
@@ -223,5 +223,5 @@
   <!-- Camera joint 1 joint -->
   <joint name="camera_joint_1_link_joint" type="revolute">
-    <limit lower="-3.14000" upper="3.14000" effort="0.00000" velocity="0.00000"/>
+    <limit lower="-3.14000" upper="3.14000" effort="10.0" velocity="3.14"/>
     <origin rpy="2.75924 -1.57080 -2.79559" xyz="-0.02297 0.00088 0.03900"/>
     <parent link="camera_joint_2_link"/>
@@ -231,5 +231,5 @@
   <!-- Camera joint 2 joint -->
   <joint name="camera_joint_2_link_joint" type="revolute">
-    <limit lower="-3.14000" upper="3.14000" effort="0.00000" velocity="0.00000"/>
+    <limit lower="-3.14000" upper="3.14000" effort="10.0" velocity="3.14"/>
     <origin rpy="3.14159 -0.00000 -3.14159" xyz="0.00665 -0.00026 -0.00516"/>
     <parent link="base_link"/>
@@ -244,6 +244,6 @@
   </joint>
   <!-- Include the gazebo materials -->
-  <xacro:include filename="$(find drone_description)/urdf/gazebo_materials.xacro"/>
+  <xacro:include filename="$(find drone_gazebo)/urdf/gazebo_materials.xacro"/>
   <!-- Include the gazebo controllers -->
-  <xacro:include filename="$(find drone_description)/urdf/drone_gazebo_controllers.xacro"/>
+  <xacro:include filename="$(find drone_gazebo_control)/urdf/drone_gazebo_controllers.xacro"/>
 </robot>

File: drone_gazebo/urdf/gazebo_materials.xacro (robot description, xacro)
@@ -1,5 +1,5 @@
 <?xml version="1.0"?>
 <robot xmlns:xacro="http://www.ros.org/wiki/xacro">
-  <!-- Main Body (Hard Plastic) -->
+  <!-- Carbon Fiber Components -->
   <gazebo reference="base_link">
     <material>
@@ -129,5 +129,5 @@
     </collision>
   </gazebo>
-  <!-- Carbon Fiber Components -->
+  <!-- Camera Joints (Hard Plastic) -->
   <gazebo reference="camera_joint_2_link">
     <material>

File: drone_gazebo_control/urdf/drone_gazebo_controllers.xacro (robot description, xacro)
@@ -42,9 +42,36 @@
       <state_interface name="effort"/>
     </joint>
+    <joint name="camera_360_link_joint">
+      <command_interface name="position">
+        <param name="min">-3.14</param>
+        <param name="max">3.14</param>
+      </command_interface>
+      <state_interface name="position"/>
+      <state_interface name="velocity"/>
+      <state_interface name="effort"/>
+    </joint>
+    <joint name="camera_joint_1_link_joint">
+      <command_interface name="position">
+        <param name="min">-3.14</param>
+        <param name="max">3.14</param>
+      </command_interface>
+      <state_interface name="position"/>
+      <state_interface name="velocity"/>
+      <state_interface name="effort"/>
+    </joint>
+    <joint name="camera_joint_2_link_joint">
+      <command_interface name="position">
+        <param name="min">-3.14</param>
+        <param name="max">3.14</param>
+      </command_interface>
+      <state_interface name="position"/>
+      <state_interface name="velocity"/>
+      <state_interface name="effort"/>
+    </joint>
   </ros2_control>
   <!-- Gazebo Plugin -->
   <gazebo>
     <plugin filename="gz_ros2_control-system" name="gz_ros2_control::GazeboSimROS2ControlPlugin">
-      <parameters>$(find drone_description)/config/drone_controllers.yaml</parameters>
+      <parameters>$(find drone_gazebo_control)/config/drone_controllers.yaml</parameters>
     </plugin>
   </gazebo>

Commit message: 🚀 feat(gazebo_plugins): Remove obsolete propulsion and aerodynamics files, add new sensor message definitions

File: drone_description/urdf/drone.urdf.xacro (robot description, xacro)
@@ -124,5 +124,5 @@
   <link name="camera_joint_1_link">
     <collision name="camera_joint_1_collision">
-    <origin rpy="0.66577 -1.57080 -0.64827" xyz="-0.00000 0.00000 0.00000"/>
+      <origin rpy="0.66577 -1.57080 -0.64827" xyz="-0.00000 0.00000 0.00000"/>
       <geometry>
         <mesh filename="package://drone_description/meshes/collisions/camera_joint1.stl" scale="0.00072 0.00072 0.00072"/>
@@ -144,5 +144,5 @@
   <link name="camera_joint_2_link">
     <collision name="camera_joint_2_collision">
-    <origin rpy="3.14159 0.00000 3.10524" xyz="0.00000 -0.00000 -0.00000"/>
+      <origin rpy="3.14159 0.00000 3.10524" xyz="0.00000 -0.00000 -0.00000"/>
       <geometry>
         <mesh filename="package://drone_description/meshes/collisions/camera_joint2.stl" scale="0.00072 0.00072 0.00072"/>
@@ -246,5 +246,5 @@
   <xacro:include filename="$(find drone_gazebo)/urdf/gazebo_materials.xacro"/>
   <!-- Include the gazebo controllers -->
-  <xacro:include filename="$(find drone_gazebo_control)/urdf/drone_gazebo_controllers.xacro"/>
+  <!-- xacro:include filename="$(find drone_gazebo_control)/urdf/drone_gazebo_controllers.xacro"/-->
   <!-- Include the gazebo plugins -->
   <xacro:include filename="$(find drone_gazebo_plugins)/urdf/drone_gazebo_plugins.xacro"/>

File: drone_gazebo_plugins/urdf/drone_gazebo_plugins.xacro (robot description, xacro)
@@ -1,8 +1,29 @@
 <?xml version="1.0"?>
 <robot xmlns:xacro="http://www.ros.org/wiki/xacro">
+  <!-- Gazebo and ROS2 bringe channel-->
   <gazebo>
-    <plugin filename="libdrone_gazebo_plugins" name="gz::sim::system::ChannelPlugin">
-      <propellers_velocity>propellers_velocity_topic</propellers_velocity>
-      <camera_360_velocity>camera_360_velocity_topic</camera_360_velocity>
+    <plugin filename="drone_gazebo_plugins" name="gz::sim::system::ChannelPlugin">
+      <propellers_velocity>propellers_velocity</propellers_velocity>
+      <camera_360_velocity>camera_360_velocity</camera_360_velocity>
+    </plugin>
+  </gazebo>
+  <!-- Gazebo odometry -->
+  <gazebo>
+    <plugin filename="gz-sim-odometry-publisher-system" name="gz::sim::system::OdometryPublisher">
+      <odom_publish_frecuency>20</odom_publish_frecuency>
+      <robot_base_frame>base_link</robot_base_frame>
+      <odom_frame>odom</odom_frame>
+    </plugin>
+  </gazebo>
+  <!-- Gazebo joint state publisher -->
+  <gazebo>
+    <plugin filename="gz-sim-joint-state-publisher-system" name="gz::sim::system::JointStatePublisher">
+      <joint_name>propeller_FL_link_joint</joint_name>
+      <joint_name>propeller_FR_link_joint</joint_name>
+      <joint_name>propeller_BL_link_joint</joint_name>
+      <joint_name>propeller_BR_link_joint</joint_name>
+      <joint_name>camera_360_link_joint</joint_name>
+      <joint_name>camera_joint_1_link_joint</joint_name>
+      <joint_name>camera_joint_2_link_joint</joint_name>
     </plugin>
   </gazebo>

Commit message: 🚀 feat(drone_gazebo_plugins): Update package dependencies and improve MAVLink integration with enhanced CMake configuration

File: drone_description/urdf/drone.urdf.xacro (robot description, xacro)
@@ -183,5 +183,4 @@
   <!-- Propeller front left joint -->
   <joint name="propeller_FL_link_joint" type="continuous">
-    <limit effort="0.3" velocity="314.16"/>
     <origin rpy="0.00000 0.00000 0.00000" xyz="-0.16748 -0.17426 0.11768"/>
     <parent link="base_link"/>
@@ -191,5 +190,4 @@
   <!-- Propeller front right joint -->
   <joint name="propeller_FR_link_joint" type="continuous">
-    <limit effort="0.3" velocity="314.16"/>
     <origin rpy="0.00000 0.00000 0.00000" xyz="-0.16745 0.17390 0.11755"/>
     <parent link="base_link"/>
@@ -199,5 +197,4 @@
   <!-- Propeller back left joint -->
   <joint name="propeller_BL_link_joint" type="continuous">
-    <limit effort="0.3" velocity="314.16"/>
     <origin rpy="0.00000 0.00000 0.00000" xyz="0.18040 -0.17426 0.11755"/>
     <parent link="base_link"/>
@@ -207,5 +204,4 @@
   <!-- Propeller back right joint -->
   <joint name="propeller_BR_link_joint" type="continuous">
-    <limit effort="0.3" velocity="314.16"/>
     <origin rpy="0.00000 0.00000 0.00000" xyz="0.18040 0.17437 0.11755"/>
     <parent link="base_link"/>

File: drone_gazebo_plugins/urdf/drone_gazebo_plugins.xacro (robot description, xacro)
@@ -11,8 +11,8 @@
   <gazebo>
     <plugin filename="gz-sim-multicopter-motor-model-system" name="gz::sim::systems::MulticopterMotorModel">
-      <robotNamespace>model/swarm_drone</robotNamespace>
-      <jointName>swarm_drone/propeller_FL_link_joint</jointName>
-      <linkName>swarm_drone/propeller_FL_link</linkName>
-      <turningDirection>cw</turningDirection>
+      <robotNamespace>swarm_drone</robotNamespace>
+      <jointName>propeller_FL_link_joint</jointName>
+      <linkName>propeller_FL_link</linkName>
+      <turningDirection>ccw</turningDirection>
       <timeConstantUp>0.0125</timeConstantUp>
       <timeConstantDown>0.025</timeConstantDown>
@@ -32,7 +32,7 @@
   <gazebo>
     <plugin filename="gz-sim-multicopter-motor-model-system" name="gz::sim::systems::MulticopterMotorModel">
-      <robotNamespace>model/swarm_drone</robotNamespace>
-      <jointName>swarm_drone/propeller_FR_link_joint</jointName>
-      <linkName>swarm_drone/propeller_FR_link</linkName>
+      <robotNamespace>swarm_drone</robotNamespace>
+      <jointName>propeller_FR_link_joint</jointName>
+      <linkName>propeller_FR_link</linkName>
       <turningDirection>ccw</turningDirection>
       <timeConstantUp>0.0125</timeConstantUp>
@@ -53,7 +53,7 @@
   <gazebo>
     <plugin filename="gz-sim-multicopter-motor-model-system" name="gz::sim::systems::MulticopterMotorModel">
-      <robotNamespace>model/swarm_drone</robotNamespace>
-      <jointName>swarm_drone/propeller_BL_link_joint</jointName>
-      <linkName>swarm_drone/propeller_BL_link</linkName>
+      <robotNamespace>swarm_drone</robotNamespace>
+      <jointName>propeller_BL_link_joint</jointName>
+      <linkName>propeller_BL_link</linkName>
       <turningDirection>ccw</turningDirection>
       <timeConstantUp>0.0125</timeConstantUp>
@@ -74,8 +74,8 @@
   <gazebo>
     <plugin filename="gz-sim-multicopter-motor-model-system" name="gz::sim::systems::MulticopterMotorModel">
-      <robotNamespace>model/swarm_drone</robotNamespace>
-      <jointName>swarm_drone/propeller_BR_link_joint</jointName>
-      <linkName>swarm_drone/propeller_BR_link</linkName>
-      <turningDirection>cw</turningDirection>
+      <robotNamespace>swarm_drone</robotNamespace>
+      <jointName>propeller_BR_link_joint</jointName>
+      <linkName>propeller_BR_link</linkName>
+      <turningDirection>ccw</turningDirection>
       <timeConstantUp>0.0125</timeConstantUp>
       <timeConstantDown>0.025</timeConstantDown>
